Commit message: Add simulated ArUco camera and marker detection pipeline
Extended the multi-robot simulation with camera frames in the robot URDF, Gazebo camera sensors, ROS-Gazebo image and camera_info bridges, and ArUco detector launch support for both robots. Added simulated ArUco marker textures and marker models to the world, then verified successful marker detection from robot_1 through /robot_1/aruco_detections. This establishes the end-to-end simulated perception pipeline needed before integrating gopigo3_aruco localization.

File: src/rosaut-gopigo3_ros2-e0b3d4594a55/gopigo3_description/urdf/gopigo3.xacro (robot description, xacro)
@@ -116,4 +116,27 @@
     </visual>
   </link>
+  <!-- ============ aruco_camera ======================== -->
+  <joint name="$(arg ns)aruco_camera_joint" type="fixed">
+    <parent link="$(arg ns)top_shelf"/>
+    <child link="$(arg ns)aruco_camera"/>
+    <!-- Camera mounted slightly forward and above the top shelf -->
+    <origin xyz="0.03 0 0.05" rpy="0 0 0"/>
+  </joint>
+  <link name="$(arg ns)aruco_camera">
+    <visual>
+      <origin xyz="0 0 0" rpy="0 0 0"/>
+      <geometry>
+        <box size="0.03 0.03 0.02"/>
+      </geometry>
+      <material name="cyan"/>
+    </visual>
+  </link>
+  <joint name="$(arg ns)aruco_camera_optical_joint" type="fixed">
+    <parent link="$(arg ns)aruco_camera"/>
+    <child link="$(arg ns)aruco_camera_optical"/>
+    <!-- ROS optical frame convention -->
+    <origin xyz="0 0 0" rpy="${-PI/2} 0 ${-PI/2}"/>
+  </joint>
+  <link name="$(arg ns)aruco_camera_optical"/>
   <!-- ============ wheels ======================== -->
   <xacro:wheel prefix="left" reflect="1.0"/>

File: src/rosaut-gopigo3_ros2-e0b3d4594a55/gopigo3_description/urdf/gopigo3_gazebo.xacro (robot description, xacro)
@@ -99,3 +99,25 @@
     </sensor>
   </gazebo>
+  <gazebo reference="$(arg ns)aruco_camera">
+    <sensor name="$(arg ns)camera_sensor" type="camera">
+      <always_on>true</always_on>
+      <update_rate>10</update_rate>
+      <visualize>true</visualize>
+      <topic>/$(arg ns)camera/image_raw</topic>
+      <camera_info_topic>/$(arg ns)camera/camera_info</camera_info_topic>
+      <gz_frame_id>$(arg ns)aruco_camera_optical</gz_frame_id>
+      <camera>
+        <horizontal_fov>1.3962634</horizontal_fov>
+        <image>
+          <width>640</width>
+          <height>480</height>
+          <format>R8G8B8</format>
+        </image>
+        <clip>
+          <near>0.05</near>
+          <far>20.0</far>
+        </clip>
+      </camera>
+    </sensor>
+  </gazebo>
 </robot>
